File: KiCad/JargonJolt/JargonJolt.kicad_sch (KiCad schematic)
At the start: 1 part, among them U1 ESP32-S3-WROOM-1-N16R2

Commit message: added jargonjolt library
Parts:
- removed U1: ESP32-S3-WROOM-1-N16R2, ESP32-S3-WROOM:XCVR_ESP32-S3-WROOM-1-N16R2, symbol ESP32-S3-WROOM-1-N16R2:ESP32-S3-WROOM-1-N16R2
- added U1: ESP32-S3-WROOM-1-N16R2, ESP32-S3-WROOM:XCVR_ESP32-S3-WROOM-1-N16R2, symbol JargonJolt:ESP32-S3-WROOM-1-N16R2
Changed lines of the file:
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@@
 (kicad_sch (version 20230121) (generator eeschema)
   (paper "A4")
-  (symbol (lib_id "ESP32-S3-WROOM-1-N16R2:ESP32-S3-WROOM-1-N16R2") (at 142.24 87.63 0) (unit 1)
+  (symbol (lib_id "JargonJolt:ESP32-S3-WROOM-1-N16R2") (at 151.13 97.79 0) (unit 1)
     (in_bom yes) (on_board yes) (dnp no) (fields_autoplaced)
-    (property "Reference" "U1" (at 142.24 49.53 0)
+    (property "Reference" "U1" (at 151.13 59.69 0)
       (effects (font (size 1.27 1.27)))
     )
-    (property "Value" "ESP32-S3-WROOM-1-N16R2" (at 142.24 52.07 0)
+    (property "Value" "ESP32-S3-WROOM-1-N16R2" (at 151.13 62.23 0)
       (effects (font (size 1.27 1.27)))
     )
-    (property "Footprint" "ESP32-S3-WROOM:XCVR_ESP32-S3-WROOM-1-N16R2" (at 142.24 87.63 0)
+    (property "Footprint" "ESP32-S3-WROOM:XCVR_ESP32-S3-WROOM-1-N16R2" (at 151.13 97.79 0)
       (effects (font (size 1.27 1.27)) (justify bottom) hide)
     )
-    (property "Datasheet" "" (at 142.24 87.63 0)
+    (property "Datasheet" "" (at 151.13 97.79 0)
       (effects (font (size 1.27 1.27)) hide)
     )
-    (property "MF" "Espressif Systems" (at 142.24 87.63 0)
+    (property "MF" "Espressif Systems" (at 151.13 97.79 0)
       (effects (font (size 1.27 1.27)) (justify bottom) hide)
     )
-    (property "MAXIMUM_PACKAGE_HEIGHT" "3.25mm" (at 142.24 87.63 0)
+    (property "MAXIMUM_PACKAGE_HEIGHT" "3.25mm" (at 151.13 97.79 0)
       (effects (font (size 1.27 1.27)) (justify bottom) hide)
     )
-    (property "Package" "NON STANDARD Espressif Systems" (at 142.24 87.63 0)
+    (property "Package" "NON STANDARD Espressif Systems" (at 151.13 97.79 0)
       (effects (font (size 1.27 1.27)) (justify bottom) hide)
     )
-    (property "Price" "None" (at 142.24 87.63 0)
+    (property "Price" "None" (at 151.13 97.79 0)
       (effects (font (size 1.27 1.27)) (justify bottom) hide)
     )
-    (property "Check_prices" "https://www.snapeda.com/parts/ESP32S3WROOM1N16R2/Espressif+Systems/view-part/?ref=eda" (at 142.24 87.63 0)
+    (property "Check_prices" "https://www.snapeda.com/parts/ESP32S3WROOM1N16R2/Espressif+Systems/view-part/?ref=eda" (at 151.13 97.79 0)
       (effects (font (size 1.27 1.27)) (justify bottom) hide)
     )
-    (property "STANDARD" "Manufacturer Recommendations" (at 142.24 87.63 0)
+    (property "STANDARD" "Manufacturer Recommendations" (at 151.13 97.79 0)
       (effects (font (size 1.27 1.27)) (justify bottom) hide)
     )
-    (property "PARTREV" "v1.0" (at 142.24 87.63 0)
+    (property "PARTREV" "v1.0" (at 151.13 97.79 0)
       (effects (font (size 1.27 1.27)) (justify bottom) hide)
     )
-    (property "SnapEDA_Link" "https://www.snapeda.com/parts/ESP32S3WROOM1N16R2/Espressif+Systems/view-part/?ref=snap" (at 142.24 87.63 0)
+    (property "SnapEDA_Link" "https://www.snapeda.com/parts/ESP32S3WROOM1N16R2/Espressif+Systems/view-part/?ref=snap" (at 151.13 97.79 0)
       (effects (font (size 1.27 1.27)) (justify bottom) hide)
     )
-    (property "MP" "ESP32S3WROOM1N16R2" (at 142.24 87.63 0)
+    (property "MP" "ESP32S3WROOM1N16R2" (at 151.13 97.79 0)
       (effects (font (size 1.27 1.27)) (justify bottom) hide)
     )
-    (property "Purchase-URL" "https://www.snapeda.com/api/url_track_click_mouser/?unipart_id=10874217&manufacturer=Espressif Systems&part_name=ESP32S3WROOM1N16R2&search_term=esp32-s3-wroom-1-n16" (at 142.24 87.63 0)
+    (property "Purchase-URL" "https://www.snapeda.com/api/url_track_click_mouser/?unipart_id=10874217&manufacturer=Espressif Systems&part_name=ESP32S3WROOM1N16R2&search_term=esp32-s3-wroom-1-n16" (at 151.13 97.79 0)
       (effects (font (size 1.27 1.27)) (justify bottom) hide)
     )
-    (property "Description" "\nBluetooth, WiFi 802.11b/g/n, Bluetooth v5.0 Transceiver Module 2.4GHz PCB Trace Surface Mount\n" (at 142.24 87.63 0)
+    (property "Description" "\nBluetooth, WiFi 802.11b/g/n, Bluetooth v5.0 Transceiver Module 2.4GHz PCB Trace Surface Mount\n" (at 151.13 97.79 0)
       (effects (font (size 1.27 1.27)) (justify bottom) hide)
     )
-    (property "Availability" "In Stock" (at 142.24 87.63 0)
+    (property "Availability" "In Stock" (at 151.13 97.79 0)
       (effects (font (size 1.27 1.27)) (justify bottom) hide)
     )
-    (property "MANUFACTURER" "Espressif" (at 142.24 87.63 0)
+    (property "MANUFACTURER" "Espressif" (at 151.13 97.79 0)
       (effects (font (size 1.27 1.27)) (justify bottom) hide)
     )
+    (pin "18")
+    (pin "35")
+    (pin "5")
+    (pin "20")
+    (pin "25")
+    (pin "10")
+    (pin "16")
+    (pin "2")
+    (pin "24")
+    (pin "27")
+    (pin "29")
+    (pin "8")
+    (pin "1")
+    (pin "3")
+    (pin "39")
+    (pin "38")
+    (pin "40")
+    (pin "26")
+    (pin "13")
+    (pin "28")
+    (pin "12")
     (pin "19")
+    (pin "4")
+    (pin "17")
+    (pin "37")
+    (pin "32")
+    (pin "6")
+    (pin "15")
+    (pin "31")
+    (pin "7")
+    (pin "33")
+    (pin "21")
+    (pin "30")
+    (pin "11")
+    (pin "23")
+    (pin "34")
+    (pin "9")
+    (pin "14")
+    (pin "36")
     (pin "22")
-    (pin "32")
-    (pin "25")
-    (pin "36")
-    (pin "39")
-    (pin "4")
-    (pin "40")
-    (pin "5")
-    (pin "7")
-    (pin "8")
-    (pin "26")
-    (pin "30")
-    (pin "13")
-    (pin "18")
-    (pin "3")
-    (pin "33")
-    (pin "12")
-    (pin "35")
-    (pin "2")
-    (pin "28")
-    (pin "6")
-    (pin "31")
-    (pin "10")
-    (pin "21")
-    (pin "23")
-    (pin "9")
-    (pin "15")
-    (pin "38")
-    (pin "29")
-    (pin "14")
-    (pin "16")
-    (pin "1")
-    (pin "27")
-    (pin "37")
-    (pin "20")
-    (pin "17")
-    (pin "34")
-    (pin "24")
-    (pin "11")
     (instances
       (project "JargonJolt"

Commit message: began working on schematic
Parts:
- removed U1: ESP32-S3-WROOM-1-N16R2, ESP32-S3-WROOM:XCVR_ESP32-S3-WROOM-1-N16R2, symbol JargonJolt:ESP32-S3-WROOM-1-N16R2
Other:
- added sheet MCU (mcu.kicad_sch)
- added sheet Memory (memory.kicad_sch)
- added sheet Power (power.kicad_sch)
- added sheet User Interface (ui.kicad_sch)
Changed lines of the file:
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@@
 (kicad_sch (version 20230121) (generator eeschema)
   (paper "A4")
-  (symbol (lib_id "JargonJolt:ESP32-S3-WROOM-1-N16R2") (at 151.13 97.79 0) (unit 1)
-    (in_bom yes) (on_board yes) (dnp no) (fields_autoplaced)
-    (property "Reference" "U1" (at 151.13 59.69 0)
-      (effects (font (size 1.27 1.27)))
+  (sheet (at 210.185 87.63) (size 23.495 10.795) (fields_autoplaced)
+    (stroke (width 0.1524) (type solid))
+    (fill (color 200 255 102 1.0000))
+    (property "Sheetname" "User Interface" (at 210.185 86.9184 0)
+      (effects (font (size 1.27 1.27)) (justify left bottom))
     )
-    (property "Value" "ESP32-S3-WROOM-1-N16R2" (at 151.13 62.23 0)
-      (effects (font (size 1.27 1.27)))
+    (property "Sheetfile" "ui.kicad_sch" (at 210.185 99.0096 0)
+      (effects (font (size 1.27 1.27)) (justify left top))
     )
-    (property "Footprint" "ESP32-S3-WROOM:XCVR_ESP32-S3-WROOM-1-N16R2" (at 151.13 97.79 0)
-      (effects (font (size 1.27 1.27)) (justify bottom) hide)
-    )
-    (property "Datasheet" "" (at 151.13 97.79 0)
-      (effects (font (size 1.27 1.27)) hide)
-    )
-    (property "MF" "Espressif Systems" (at 151.13 97.79 0)
-      (effects (font (size 1.27 1.27)) (justify bottom) hide)
-    )
-    (property "MAXIMUM_PACKAGE_HEIGHT" "3.25mm" (at 151.13 97.79 0)
-      (effects (font (size 1.27 1.27)) (justify bottom) hide)
-    )
-    (property "Package" "NON STANDARD Espressif Systems" (at 151.13 97.79 0)
-      (effects (font (size 1.27 1.27)) (justify bottom) hide)
-    )
-    (property "Price" "None" (at 151.13 97.79 0)
-      (effects (font (size 1.27 1.27)) (justify bottom) hide)
-    )
-    (property "Check_prices" "https://www.snapeda.com/parts/ESP32S3WROOM1N16R2/Espressif+Systems/view-part/?ref=eda" (at 151.13 97.79 0)
-      (effects (font (size 1.27 1.27)) (justify bottom) hide)
-    )
-    (property "STANDARD" "Manufacturer Recommendations" (at 151.13 97.79 0)
-      (effects (font (size 1.27 1.27)) (justify bottom) hide)
-    )
-    (property "PARTREV" "v1.0" (at 151.13 97.79 0)
-      (effects (font (size 1.27 1.27)) (justify bottom) hide)
-    )
-    (property "SnapEDA_Link" "https://www.snapeda.com/parts/ESP32S3WROOM1N16R2/Espressif+Systems/view-part/?ref=snap" (at 151.13 97.79 0)
-      (effects (font (size 1.27 1.27)) (justify bottom) hide)
-    )
-    (property "MP" "ESP32S3WROOM1N16R2" (at 151.13 97.79 0)
-      (effects (font (size 1.27 1.27)) (justify bottom) hide)
-    )
-    (property "Purchase-URL" "https://www.snapeda.com/api/url_track_click_mouser/?unipart_id=10874217&manufacturer=Espressif Systems&part_name=ESP32S3WROOM1N16R2&search_term=esp32-s3-wroom-1-n16" (at 151.13 97.79 0)
-      (effects (font (size 1.27 1.27)) (justify bottom) hide)
-    )
-    (property "Description" "\nBluetooth, WiFi 802.11b/g/n, Bluetooth v5.0 Transceiver Module 2.4GHz PCB Trace Surface Mount\n" (at 151.13 97.79 0)
-      (effects (font (size 1.27 1.27)) (justify bottom) hide)
-    )
-    (property "Availability" "In Stock" (at 151.13 97.79 0)
-      (effects (font (size 1.27 1.27)) (justify bottom) hide)
-    )
-    (property "MANUFACTURER" "Espressif" (at 151.13 97.79 0)
-      (effects (font (size 1.27 1.27)) (justify bottom) hide)
-    )
-    (pin "18")
-    (pin "35")
-    (pin "5")
-    (pin "20")
-    (pin "25")
-    (pin "10")
-    (pin "16")
-    (pin "2")
-    (pin "24")
-    (pin "27")
-    (pin "29")
-    (pin "8")
-    (pin "1")
-    (pin "3")
-    (pin "39")
-    (pin "38")
-    (pin "40")
-    (pin "26")
-    (pin "13")
-    (pin "28")
-    (pin "12")
-    (pin "19")
-    (pin "4")
-    (pin "17")
-    (pin "37")
-    (pin "32")
-    (pin "6")
-    (pin "15")
-    (pin "31")
-    (pin "7")
-    (pin "33")
-    (pin "21")
-    (pin "30")
-    (pin "11")
-    (pin "23")
-    (pin "34")
-    (pin "9")
-    (pin "14")
-    (pin "36")
-    (pin "22")
     (instances
       (project "JargonJolt"
-        (path "/39fa52d1-bab8-41e3-aba2-e2f783adaf1f"
-          (reference "U1") (unit 1)
-        )
+        (path "/39fa52d1-bab8-41e3-aba2-e2f783adaf1f" (page "4"))
       )
     )
+  )
+  (sheet (at 63.5 106.68) (size 19.685 17.78) (fields_autoplaced)
+    (stroke (width 0.1524) (type solid))
+    (fill (color 113 64 255 1.0000))
+    (property "Sheetname" "Memory" (at 63.5 105.9684 0)
+      (effects (font (size 1.27 1.27)) (justify left bottom))
+    )
+    (property "Sheetfile" "memory.kicad_sch" (at 63.5 125.0446 0)
+      (effects (font (size 1.27 1.27)) (justify left top))
+    )
+    (instances
+      (project "JargonJolt"
+        (path "/39fa52d1-bab8-41e3-aba2-e2f783adaf1f" (page "5"))
+      )
+    )
+  )
+  (sheet (at 118.745 114.3) (size 23.495 7.62) (fields_autoplaced)
+    (stroke (width 0.1524) (type solid))
+    (fill (color 255 94 97 1.0000))
+    (property "Sheetname" "Power" (at 118.745 113.5884 0)
+      (effects (font (size 1.27 1.27)) (justify left bottom))
+    )
+    (property "Sheetfile" "power.kicad_sch" (at 118.745 122.5046 0)
+      (effects (font (size 1.27 1.27)) (justify left top))
+    )
+    (instances
+      (project "JargonJolt"
+        (path "/39fa52d1-bab8-41e3-aba2-e2f783adaf1f" (page "3"))
+      )
+    )
+  )
+  (sheet (at 111.76 67.31) (size 35.56 24.765) (fields_autoplaced)
+    (stroke (width 0.1524) (type solid))
+    (fill (color 91 138 255 1.0000))
+    (property "Sheetname" "MCU" (at 111.76 66.5984 0)
+      (effects (font (size 1.27 1.27)) (justify left bottom))
+    )
+    (property "Sheetfile" "mcu.kicad_sch" (at 111.76 92.6596 0)
+      (effects (font (size 1.27 1.27)) (justify left top))
+    )
+    (instances
+      (project "JargonJolt"
+        (path "/39fa52d1-bab8-41e3-aba2-e2f783adaf1f" (page "2"))
+      )
+    )

Commit message: worked on pinout
Other:
- sheet MCU ports: added BUTTON1, BUTTON2, BUTTON3, VSPI_CS1, VSPI_CS2, VSPI_MISO, VSPI_MOSI, VSPI_SCLK; removed none
- sheet Memory ports: added VSPI_CS1, VSPI_CS2, VSPI_MISO, VSPI_MOSI, VSPI_SCLK; removed none
- sheet User Interface ports: added BUTTON1, BUTTON2, BUTTON3; removed none
Changed lines of the file:
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@@
 (kicad_sch (version 20230121) (generator eeschema)
   (paper "A4")
-  (sheet (at 210.185 87.63) (size 23.495 10.795) (fields_autoplaced)
+  (wire (pts (xy 107.061 86.106) (xy 111.76 86.106))
+    (stroke (width 0) (type default))
+  )
+  (wire (pts (xy 83.312 117.348) (xy 111.76 117.348))
+    (stroke (width 0) (type default))
+  )
+  (wire (pts (xy 83.185 114.681) (xy 109.347 114.681))
+    (stroke (width 0) (type default))
+  )
+  (wire (pts (xy 83.185 112.395) (xy 107.061 112.395))
+    (stroke (width 0) (type default))
+  )
+  (wire (pts (xy 147.32 90.678) (xy 165.608 90.678))
+    (stroke (width 0) (type default))
+  )
+  (wire (pts (xy 109.347 114.681) (xy 109.347 88.011))
+    (stroke (width 0) (type default))
+  )
+  (wire (pts (xy 147.32 85.979) (xy 165.608 85.979))
+    (stroke (width 0) (type default))
+  )
+  (wire (pts (xy 107.061 112.395) (xy 107.061 86.106))
+    (stroke (width 0) (type default))
+  )
+  (wire (pts (xy 104.902 83.566) (xy 111.76 83.566))
+    (stroke (width 0) (type default))
+  )
+  (wire (pts (xy 147.32 88.392) (xy 165.608 88.392))
+    (stroke (width 0) (type default))
+  )
+  (wire (pts (xy 83.058 110.363) (xy 104.902 110.363))
+    (stroke (width 0) (type default))
+  )
+  (wire (pts (xy 109.347 88.011) (xy 111.76 88.011))
+    (stroke (width 0) (type default))
+  )
+  (wire (pts (xy 111.76 117.348) (xy 111.76 90.17))
+    (stroke (width 0) (type default))
+  )
+  (wire (pts (xy 104.902 110.363) (xy 104.902 83.566))
+    (stroke (width 0) (type default))
+  )
+  (sheet (at 165.608 79.756) (size 23.495 11.938) (fields_autoplaced)
     (stroke (width 0.1524) (type solid))
     (fill (color 200 255 102 1.0000))
-    (property "Sheetname" "User Interface" (at 210.185 86.9184 0)
+    (property "Sheetname" "User Interface" (at 165.608 79.0444 0)
       (effects (font (size 1.27 1.27)) (justify left bottom))
     )
-    (property "Sheetfile" "ui.kicad_sch" (at 210.185 99.0096 0)
+    (property "Sheetfile" "ui.kicad_sch" (at 165.608 92.2786 0)
       (effects (font (size 1.27 1.27)) (justify left top))
+    )
+    (pin "BUTTON1" input (at 165.608 85.979 180)
+      (effects (font (size 1.27 1.27)) (justify left))
+    )
+    (pin "BUTTON2" input (at 165.608 88.392 180)
+      (effects (font (size 1.27 1.27)) (justify left))
+    )
+    (pin "BUTTON3" input (at 165.608 90.678 180)
+      (effects (font (size 1.27 1.27)) (justify left))
     )
     (instances
@@
     (property "Sheetfile" "memory.kicad_sch" (at 63.5 125.0446 0)
       (effects (font (size 1.27 1.27)) (justify left top))
+    )
+    (pin "VSPI_CS1" input (at 83.185 110.49 0)
+      (effects (font (size 1.27 1.27)) (justify right))
+    )
+    (pin "VSPI_MOSI" input (at 83.185 112.522 0)
+      (effects (font (size 1.27 1.27)) (justify right))
+    )
+    (pin "VSPI_MISO" input (at 83.185 114.808 0)
+      (effects (font (size 1.27 1.27)) (justify right))
+    )
+    (pin "VSPI_CS2" input (at 83.185 108.077 0)
+      (effects (font (size 1.27 1.27)) (justify right))
+    )
+    (pin "VSPI_SCLK" input (at 83.185 117.348 0)
+      (effects (font (size 1.27 1.27)) (justify right))
     )
     (instances
@@
       (effects (font (size 1.27 1.27)) (justify left top))
     )
+    (pin "BUTTON1" input (at 147.32 85.979 0)
+      (effects (font (size 1.27 1.27)) (justify right))
+    )
+    (pin "BUTTON2" input (at 147.32 88.392 0)
+      (effects (font (size 1.27 1.27)) (justify right))
+    )
+    (pin "VSPI_MOSI" input (at 111.76 86.106 180)
+      (effects (font (size 1.27 1.27)) (justify left))
+    )
+    (pin "VSPI_SCLK" input (at 111.76 90.17 180)
+      (effects (font (size 1.27 1.27)) (justify left))
+    )
+    (pin "VSPI_MISO" input (at 111.76 88.011 180)
+      (effects (font (size 1.27 1.27)) (justify left))
+    )
+    (pin "VSPI_CS1" input (at 111.76 83.566 180)
+      (effects (font (size 1.27 1.27)) (justify left))
+    )
+    (pin "VSPI_CS2" input (at 111.76 81.28 180)
+      (effects (font (size 1.27 1.27)) (justify left))
+    )
+    (pin "BUTTON3" input (at 147.32 90.678 0)
+      (effects (font (size 1.27 1.27)) (justify right))
+    )
     (instances
